File: kicad-proj/s1-ecg-demo.sch (KiCad schematic (older format))
At the start: 58 parts, among them J1 Left arm, J2 Right arm, J3 Right leg, J4 USB-C-16-Pin, J5 TC2030, J6 Current Probe, J7 Battery Port, U1 AD8233

Commit message: Final files ready for order
Parts:
- removed R13: 100k, Resistor_SMD:R_0201_0603Metric, symbol Device:R_Small
- C1: renamed from C5; value 0.22u -> 220nF
- C2: renamed from C1; value 0.22u -> 220nF
- C3: renamed from C7; value 1u -> 1uF
- C4: renamed from C3; value 1n -> 1nF
- C5: renamed from C6; value 0.1u -> 100nF
- C6: renamed from C8; value 10u -> 10uF
- C7: renamed from C4; value 22n -> 22nF
- C8: renamed from C2; value 10n -> 10nF
- J2: renamed from J5; Note (none) -> Debug Port
- R16: renamed from R4; value 665 -> 665R
- R17: renamed from R6; value 665 -> 665R
- R18: renamed from R14; value 665 -> 665R
- R19: renamed from R15; value 665 -> 665R
- R20: renamed from R16; value 665 -> 665R
- R21: renamed from R17; value 665 -> 665R
- R22: renamed from R20; value 665 -> 665R
- U1: footprint s1-ecg-demo:WLCSP-20 -> s1-ecg-demo:WLCSP-20-no-paste
- renumbered J2 to J3, J3 to J4, J6 to J5, J4 to J6, R18 to R1, R1 to R11, R7 to R12, R8 to R13, R22 to R14, R23 to R15, R11 to R2, R12 to R3, R19 to R4, R9 to R6, R21 to R7, R3 to R8, R2 to R9
Connections:
- net GND: now also J6.A1/B12 (GND), J6.A12/B1 (GND)
- net at C1.2, U1.A4 (HPSENSE): now also R1.2; no longer R1.1
- net at C2.2, U1.B4 (IAOUT): now also R1.1; no longer R1.2
- net at C7.1, R12.1, U1.C3 (REFOUT): now also R11.1; no longer R11.2
- net at U1.D4 (SW): now also C2.1, R11.2, R9.1
- net at J6.A5 (CC1): now also R14.2
- net at J6.B5 (CC2): now also R15.2
- net ECG_OUT renamed ecg-out
- net LED1 renamed led1
- net LED2 renamed led2
- net LED3 renamed led3
- net LED4 renamed led4
- net LED5 renamed led5
- net LED6 renamed led6
- net LED7 renamed led7
- net LOD renamed lead-detect
- net VBAT renamed Vbatt
- net ~SDN renamed ~shutdown
- no-connect marks 10 -> 6
Other:
- note added: "Cut JP1 for current\nmeasurement"
- moved on the sheet: C1, C2, C3, C4, C5, C6, C7, C8, J1, J3, J4, J5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

Commit message: Added shutdown pullup resistor Adjusted current probe header location Updated BOM Exported v2 gerber
Parts:
- added R3: 10M, Resistor_SMD:R_0201_0603Metric, symbol Device:R_Small
- renumbered R9 to R10, R10 to R11, R11 to R12, R12 to R13, R13 to R14, R14 to R15, R15 to R16, R16 to R17, R17 to R18, R18 to R19, R19 to R20, R20 to R21, R21 to R22, R22 to R23, R3 to R4, R4 to R5, R5 to R6, R6 to R7, R7 to R8, R8 to R9
Connections:
- net +1V8: now also R3.1
- net ~shutdown: now also R3.2
Other:
- moved on the sheet: J2, MOD1

Commit message: Fixed ground break Isolation around battery positive terminal Removed the cuttable jumper Cleaned up silkscreen Added 0.1" pin jumper to BOM
Parts:
- removed JP1: Jumper_NC_Small, Jumper:SolderJumper-2_P1.3mm_Bridged_RoundedPad1.0x1.5mm, symbol Device:Jumper_NC_Small
- J5: value Current Probe -> Current Measure
Other:
- note added: "Remove jumper to\nmeasure current\nacross this header."
- note removed: "Cut JP1 for current\nmeasurement"
Changed lines of the file:
@@
 Vusb
-$Comp
-L Device:Jumper_NC_Small JP1
-U 1 1 611AAD4D
-P 9900 5000
-F 0 "JP1" H 9900 4907 50  0000 C CNN
-F 1 "Jumper_NC_Small" V 9855 4953 50  0001 R CNN
-F 2 "Jumper:SolderJumper-2_P1.3mm_Bridged_RoundedPad1.0x1.5mm" H 9900 5000 50  0001 C CNN
-F 3 "~" H 9900 5000 50  0001 C CNN
-	1    9900 5000
-	-1   0    0    -1
-$EndComp
 $Comp
 L Mechanical:Fiducial FID1
@@
 F 3 "~" H 6150 7150 50  0001 C CNN
 	1    6150 7150
-	1    0    0    -1
-$EndComp
-$Comp
-L s1-ecg-demo:TC2030 J2
-U 1 1 6118E478
-P 10000 2300
-F 0 "J2" H 10228 2641 50  0000 L CNN
-F 1 "TC2030" H 10228 2550 50  0000 L CNN
-F 2 "Connector:Tag-Connect_TC2030-IDC-NL_2x03_P1.27mm_Vertical" H 8200 3000 50  0001 C CNN
-F 3 "" H 8200 3000 50  0001 C CNN
-F 4 "Debug Port" H 10228 2459 50  0000 L CNN "Note"
-	1    10000 2300
 	1    0    0    -1
 $EndComp
@@
 Wire Wire Line
 	8850 2500 8800 2500
-Wire Wire Line
-	9750 5000 9750 4900
-Wire Wire Line
-	9750 5000 9800 5000
-Wire Wire Line
-	9750 4900 10100 4900
 $Comp
 L Connector_Generic:Conn_01x02 J5
@@
 P 10300 4900
 F 0 "J5" H 10380 4892 50  0000 L CNN
-F 1 "Current Probe" H 10380 4801 50  0000 L CNN
+F 1 "Current Measure" H 10380 4801 50  0000 L CNN
 F 2 "s1-ecg-demo:Conn_2_SMD_2.54mm" H 10300 4900 50  0001 C CNN
 F 3 "~" H 10300 4900 50  0001 C CNN
@@
 $EndComp
 Wire Wire Line
-	10000 5000 10050 5000
-Wire Wire Line
 	10050 5000 10050 5300
 Wire Wire Line
 	10050 5300 10100 5300
-Connection ~ 10050 5000
 Wire Wire Line
 	10050 5000 10100 5000
@@
 	-1   0    0    1
 $EndComp
-Text Notes 9950 5300 2    50   ~ 0
-Cut JP1 for current\nmeasurement
-Wire Wire Line
-	9650 4900 9750 4900
-Connection ~ 9750 4900
+Text Notes 10250 4800 0    50   ~ 0
+Remove jumper to\nmeasure current\nacross this header.
 $Comp
 L Device:R_Small R3
@@
 Wire Wire Line
 	7000 2500 7800 2500
+Wire Wire Line
+	9650 4900 10100 4900
+$Comp
+L s1-ecg-demo:TC2030 J2
+U 1 1 6118E478
+P 10000 2300
+F 0 "J2" H 10228 2641 50  0000 L CNN
+F 1 "TC2030" H 10228 2550 50  0000 L CNN
+F 2 "Connector:Tag-Connect_TC2030-IDC-NL_2x03_P1.27mm_Vertical" H 8200 3000 50  0001 C CNN
+F 3 "" H 8200 3000 50  0001 C CNN
+F 4 "Debug Port" H 10228 2459 50  0000 L CNN "Note"
+	1    10000 2300
+	1    0    0    -1
+$EndComp
 $EndSCHEMATC
